Commit message: driving to block works

File: me326_locobot_group5/model/blue_cube.urdf (robot description, URDF)
Before this commit: robot blue_cube, 1 links, 0 joints
Links:
- link my_box: mass 0.5 -> 0.05

File: me326_locobot_group5/model/green_cube.urdf (robot description, URDF)
Before this commit: robot green_cube, 1 links, 0 joints
Links:
- link my_box: mass 0.5 -> 0.05

File: me326_locobot_group5/model/red_cube.urdf (robot description, URDF)
Before this commit: robot red_cube, 1 links, 0 joints
Links:
- link my_box: mass 0.5 -> 0.05

File: me326_locobot_group5/model/yellow_cube.urdf (robot description, URDF)
Before this commit: robot yellow_cube, 1 links, 0 joints
Links:
- link my_box: mass 0.5 -> 0.05

Commit message: fixed bounding box

File: me326_locobot_group5/model/blue_cube.urdf (robot description, URDF)
Before this commit: robot blue_cube, 1 links, 0 joints
Links:
- link my_box: mass 0.05 -> 0.005

File: me326_locobot_group5/model/green_cube.urdf (robot description, URDF)
Before this commit: robot green_cube, 1 links, 0 joints
Links:
- link my_box: mass 0.05 -> 0.005

File: me326_locobot_group5/model/red_cube.urdf (robot description, URDF)
Before this commit: robot red_cube, 1 links, 0 joints
Links:
- link my_box: mass 0.05 -> 0.005

File: me326_locobot_group5/model/yellow_cube.urdf (robot description, URDF)
Before this commit: robot yellow_cube, 1 links, 0 joints
Links:
- link my_box: mass 0.05 -> 0.005

Commit message: fixed cube inertias

File: me326_locobot_group5/model/blue_cube.urdf (robot description, URDF)
Before this commit: robot blue_cube, 1 links, 0 joints
Links:
- link my_box: mass 0.005 -> 0.05

File: me326_locobot_group5/model/green_cube.urdf (robot description, URDF)
Before this commit: robot green_cube, 1 links, 0 joints
Links:
- link my_box: mass 0.005 -> 0.05

File: me326_locobot_group5/model/red_cube.urdf (robot description, URDF)
Before this commit: robot red_cube, 1 links, 0 joints
Links:
- link my_box: mass 0.005 -> 0.05

File: me326_locobot_group5/model/yellow_cube.urdf (robot description, URDF)
Before this commit: robot yellow_cube, 1 links, 0 joints
Links:
- link my_box: mass 0.005 -> 0.05
